File: BRIDGE.kicad_sch (KiCad schematic)
At the start: 14 parts, among them Q5 SWHA088R06VT, Q6 SWHA088R06VT, U4 DGD0506A, U5 INA199B2DCK

Commit message: なにか変えた
Parts:
- added R23, R24: 10k, Resistor_SMD:R_0603_1608Metric_Pad0.98x0.95mm_HandSolder, symbol Device:R
- U5: value INA199B2DCK -> INA199x1DCK
- renumbered R7 to R9
Connections:
- net +3.3V: now also R23.1
- net GND: now also R24.2; no longer U5.1 (REF)
- new net: R23.2, R24.1, U5.1 (REF)
Other:
- moved on the sheet: C14, R9
