File: CAN.kicad_sch (KiCad schematic)
At the start: 4 parts, among them U11 MCP2551-I-SN

Commit message: なにか変えた
Parts:
- renumbered JP2 to JP4, R18 to R26
Changed lines of the file:
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@@
   (symbol (lib_id "Jumper:Jumper_3_Open") (at 111.76 95.25 90) (unit 1)
     (in_bom yes) (on_board yes) (dnp no) (fields_autoplaced)
-    (property "Reference" "JP2" (at 109.22 94.615 90)
+    (property "Reference" "JP4" (at 109.22 94.615 90)
       (effects (font (size 1.27 1.27)) (justify left))
     )
@@
       (project "sMDU"
         (path "/01e9384d-acb3-40ee-83e0-c5c8a07f30ec/8ffda33b-906e-48a0-9f0c-e538c562559b"
-          (reference "JP2") (unit 1)
+          (reference "JP4") (unit 1)
         )
       )
@@
   (symbol (lib_id "power:GND") (at 111.76 101.6 0) (unit 1)
     (in_bom yes) (on_board yes) (dnp no) (fields_autoplaced)
-    (property "Reference" "#PWR062" (at 111.76 107.95 0)
+    (property "Reference" "#PWR070" (at 111.76 107.95 0)
       (effects (font (size 1.27 1.27)) hide)
     )
@@
       (project "sMDU"
         (path "/01e9384d-acb3-40ee-83e0-c5c8a07f30ec/8ffda33b-906e-48a0-9f0c-e538c562559b"
-          (reference "#PWR062") (unit 1)
+          (reference "#PWR070") (unit 1)
         )
       )
@@
   (symbol (lib_id "power:GND") (at 128.27 102.87 0) (unit 1)
     (in_bom yes) (on_board yes) (dnp no) (fields_autoplaced)
-    (property "Reference" "#PWR063" (at 128.27 109.22 0)
+    (property "Reference" "#PWR071" (at 128.27 109.22 0)
       (effects (font (size 1.27 1.27)) hide)
     )
@@
       (project "sMDU"
         (path "/01e9384d-acb3-40ee-83e0-c5c8a07f30ec/8ffda33b-906e-48a0-9f0c-e538c562559b"
-          (reference "#PWR063") (unit 1)
+          (reference "#PWR071") (unit 1)
         )
       )
@@
   (symbol (lib_id "Device:R") (at 162.56 92.71 90) (unit 1)
     (in_bom yes) (on_board yes) (dnp no) (fields_autoplaced)
-    (property "Reference" "R18" (at 162.56 87.63 90)
+    (property "Reference" "R26" (at 162.56 87.63 90)
       (effects (font (size 1.27 1.27)))
     )
@@
       (project "sMDU"
         (path "/01e9384d-acb3-40ee-83e0-c5c8a07f30ec/8ffda33b-906e-48a0-9f0c-e538c562559b"
-          (reference "R18") (unit 1)
+          (reference "R26") (unit 1)
         )
       )
@@
   (symbol (lib_id "power:+5V") (at 111.76 88.9 0) (unit 1)
     (in_bom yes) (on_board yes) (dnp no) (fields_autoplaced)
-    (property "Reference" "#PWR061" (at 111.76 92.71 0)
+    (property "Reference" "#PWR069" (at 111.76 92.71 0)
       (effects (font (size 1.27 1.27)) hide)
     )
@@
       (project "sMDU"
         (path "/01e9384d-acb3-40ee-83e0-c5c8a07f30ec/8ffda33b-906e-48a0-9f0c-e538c562559b"
-          (reference "#PWR061") (unit 1)
+          (reference "#PWR069") (unit 1)
         )
       )
@@
   (symbol (lib_id "power:+5V") (at 142.24 77.47 0) (unit 1)
     (in_bom yes) (on_board yes) (dnp no) (fields_autoplaced)
-    (property "Reference" "#PWR064" (at 142.24 81.28 0)
+    (property "Reference" "#PWR072" (at 142.24 81.28 0)
       (effects (font (size 1.27 1.27)) hide)
     )
@@
       (project "sMDU"
         (path "/01e9384d-acb3-40ee-83e0-c5c8a07f30ec/8ffda33b-906e-48a0-9f0c-e538c562559b"
-          (reference "#PWR064") (unit 1)
+          (reference "#PWR072") (unit 1)
         )
       )
@@
   (symbol (lib_id "power:GND") (at 142.24 102.87 0) (unit 1)
     (in_bom yes) (on_board yes) (dnp no) (fields_autoplaced)
-    (property "Reference" "#PWR065" (at 142.24 109.22 0)
+    (property "Reference" "#PWR073" (at 142.24 109.22 0)
       (effects (font (size 1.27 1.27)) hide)
     )
@@
       (project "sMDU"
         (path "/01e9384d-acb3-40ee-83e0-c5c8a07f30ec/8ffda33b-906e-48a0-9f0c-e538c562559b"
-          (reference "#PWR065") (unit 1)
+          (reference "#PWR073") (unit 1)
         )
       )
@@
   (symbol (lib_id "power:GND") (at 168.91 85.09 0) (unit 1)
     (in_bom yes) (on_board yes) (dnp no)
-    (property "Reference" "#PWR066" (at 168.91 91.44 0)
+    (property "Reference" "#PWR074" (at 168.91 91.44 0)
       (effects (font (size 1.27 1.27)) hide)
     )
@@
       (project "sMDU"
         (path "/01e9384d-acb3-40ee-83e0-c5c8a07f30ec/8ffda33b-906e-48a0-9f0c-e538c562559b"
-          (reference "#PWR066") (unit 1)
-        )
-      )
+          (reference "#PWR074") (unit 1)
+        )
+      )
