File: MCU.kicad_sch (KiCad schematic)
At the start: 7 parts, among them J1 Conn_01x04, U6 STM32F303K8Tx, Y1 Resonator

Commit message: なにか変えた
Connections:
- net RM_ENC2: now reaches U6.10 (PA4)
- net I2C_SCL: now reaches U6.25 (PA15)
- net RM_ENC1: now reaches U6.9 (PA3)
- net SWCLK renamed I2C_SDA
- no-connect marks 3 -> 0
Other:
- note added: "LED RGB:TMR2 CH1,2,3 PWM:TMR1 CH1,2,3 BATT_V:ADC2 CH2 U_I:ADC2 CH3 V_I:ADC2 CH4 W_I:ADC1 CH11 Robotmaster motor H1:ADC2 CH1 Robotmaster motor H2:ADC1 CH4 PB3:SPI SCK PB4:SPI MISO / TMR3 CH1 PB5:SPI SS / TMR3 CH2"
- note removed: "LED RGB:TMR2 CH1,2,3 PWM:TMR1 CH1,2,3 BATT_V:ADC2 CH2 U_I:ADC2 CH3 V_I:ADC2 CH4 W_I:ADC1 CH11 PB3:SPI SCK PB4:SPI MISO / TMR3 CH1 PB5:SPI SS / TMR3 CH2"
