File: sMDU.kicad_pcb (KiCad board)
At the start: 4 copper layers, 77.6 x 30.1 mm, 85 parts, among them J1 Conn_01x04, J2 USB_C_Receptacle_USB2.0, Q1 BSC050N04LS, Q2 BSC050N04LS, Q3 BSC050N04LS, Q4 BSC050N04LS, Q5 BSC050N04LS, Q6 BSC050N04LS, U1 9V_LR, U10 INA199xxDCK, U11 MCP2551-I-SN, U12 CH340E, U13 XC6206PxxxMR, U2 L78L05_SOT89, U4 DGD0506A, U5 INA199xxDCK, U6 STM32F303K8Tx, U7 DGD0506A, U8 INA199xxDCK, U9 DGD0506A, Y1 Resonator

Commit message: なにか変えた
Parts:
- added R16: 10k, Resistor_SMD:R_0603_1608Metric_Pad0.98x0.95mm_HandSolder, F.Cu at (188.6, 78.4)
- added R17: 10k, Resistor_SMD:R_0603_1608Metric_Pad0.98x0.95mm_HandSolder, F.Cu at (185.0, 75.8)
- added R23: 10k, Resistor_SMD:R_0603_1608Metric_Pad0.98x0.95mm_HandSolder, F.Cu at (152.5, 114.2)
- added R24: 10k, Resistor_SMD:R_0603_1608Metric_Pad0.98x0.95mm_HandSolder, F.Cu at (152.5, 116.7)
- added R7: 10k, Resistor_SMD:R_0603_1608Metric_Pad0.98x0.95mm_HandSolder, F.Cu at (169.0, 74.3)
- added R8: 10k, Resistor_SMD:R_0603_1608Metric_Pad0.98x0.95mm_HandSolder, F.Cu at (170.6, 74.3)
- JP1: value Jumper_3_Open -> C2P
- Q1, Q2, Q3, Q4, Q5, Q6: value BSC050N04LS -> SWHA088R06VT
- U10, U5, U8: value INA199xxDCK -> INA199x1DCK
- moved U6 0.58 mm to (123.9, 88.1)
- moved C16 0.43 mm to (130.9, 87.8)
- moved Y1 0.19 mm to (117.3, 92.2)
- moved C15 0.15 mm to (119.6, 94.6)
- renumbered JP2 to JP4, R8 to R12, R9 to R13, R10 to R14, R11 to R15, R12 to R18, R13 to R19, R14 to R20, R15 to R21, R16 to R22, R17 to R25, R18 to R26, R19 to R27, R20 to R28, R7 to R9, U13 to U3
Connections:
- ENC1 pad 3: /MCU/PB4 -> /MCU/SWCLK
- ENC1 pad 4: /MCU/PB3 -> /MCU/I2C_SCL
- U10 pad 1: GND -> Net-(U10-REF)
- U5 pad 1: GND -> Net-(U5-REF)
- U6 pad 10: unconnected-(U6-PA4-Pad10) -> /MCU/SWCLK
- U6 pad 25: unconnected-(U6-PA15-Pad25) -> /MCU/I2C_SCL
- U6 pad 26: /MCU/PB3 -> /MCU/I2C_SCL
- U6 pad 27: /MCU/PB4 -> /MCU/SWCLK
- U6 pad 9: unconnected-(U6-PA3-Pad9) -> /MCU/PB5
- U8 pad 1: GND -> Net-(U8-REF)
Routing:
- net +3.3V: track 177.5 -> 196.0 mm
- net /MCU/I2C_SCL: track 0.00 -> 12.3 mm
- net /MCU/SWCLK: track 24.6 -> 36.4 mm
- net /MCU/PB3: track 11.8 -> 0.00 mm
- net /MCU/PB4: track 10.5 -> 0.00 mm
- net /BRIDGE/PWM: track 22.0 -> 12.2 mm
- net /BRIDGE1/PWM: track 23.9 -> 14.4 mm
- net Net-(U5-REF): track 0.00 -> 4.18 mm
- net GND: track 120.9 -> 117.5 mm
- net /MCU/SWDIO: track 27.8 -> 30.8 mm
- net /BRIDGE2/PWM: track 32.5 -> 30.0 mm
- net /MCU/NRST: track 29.4 -> 31.6 mm
- net /MCU/LED_R: track 15.6 -> 14.9 mm
- net /MCU/LED_G: track 15.9 -> 15.2 mm
- net /MCU/LED_B: track 15.9 -> 15.3 mm
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