File: sMDU.kicad_sch (KiCad schematic)
At the start: 26 parts, among them U1 9V_LR, U13 XC6206PxxxMR, U2 L78L05_SOT89

Commit message: なにか変えた
Parts:
- JP1: value Jumper_3_Open -> C2P
- renumbered U13 to U3
Connections:
- net MCU/PB3 renamed MCU/I2C_SCL
- net MCU/PB4 renamed MCU/I2C_SDA
Other:
- sheet MCU ports: added I2C_SCL, I2C_SDA, RM_ENC1, RM_ENC2; removed none
- moved on the sheet: ENC1, JP1
